File: Lark1 Flight computer/Lark1/Lark1.kicad_sch (KiCad schematic)
At the start: 3 parts, among them J1 Screw_Terminal_01x02, SW1 SW_SPDT, U1 esp32_38_pins dev board

Commit message: Lark1 almost done, indicators left
Parts:
- added J2, J3, J4, J5: Screw_Terminal_01x02, symbol Connector:Screw_Terminal_01x02
- added Q1, Q2, Q3, Q4: IRLZ44N, Package_TO_SOT_THT:TO-220-3_Vertical, symbol Transistor_FET:IRLZ44N
- added R1, R2, R3, R4: 10k, symbol Device:R
- added U2: module_mpu6050, usini_sensors:module_mpu6050, symbol usini_sensors:module_mpu6050
Connections:
- net +3.3V: now also U1.19 (5V), J2.2 (Pin_2), J3.2 (Pin_2), J4.2 (Pin_2), J5.2 (Pin_2)
- net GND: now also U1.38 (GND), Q1.3 (S), Q2.3 (S), Q3.3 (S), Q4.3 (S), R1.2, R2.2, R3.2, R4.2, U2.2 (GND)
- net 3v3_esp32: now reaches U1.1 (3.3V)
- net 3v3_esp32: now also U2.1 (VCC)
- net M4_PWM: now reaches U1.28 (GPIO17)
- net M4_PWM: now also Q4.1 (G), R4.1
- net M3_PWM: now reaches U1.29 (GPIO5)
- net M3_PWM: now also Q3.1 (G), R3.1
- net M2_PWM: now reaches U1.30 (GPIO18)
- net M2_PWM: now also Q2.1 (G), R2.1
- net M1_PWM: now reaches U1.31 (GPIO19)
- net M1_PWM: now also Q1.1 (G), R1.1
- net MPU6050_SDA: now reaches U1.33 (GPIO21)
- net MPU6050_SDA: now also U2.4 (SDA)
- net MPU6050_SCL: now reaches U1.36 (GPIO22)
- net MPU6050_SCL: now also U2.3 (SCL)
- new net M1_GND: J2.1 (Pin_1), Q1.2 (D)
- new net M2_GND: J3.1 (Pin_1), Q2.2 (D)
- new net M3_GND: J4.1 (Pin_1), Q3.2 (D)
- new net M4_GND: J5.1 (Pin_1), Q4.2 (D)
Other:
- moved on the sheet: U1

Commit message: Lark1 1.0
Parts:
- added BZ1: Buzzer, symbol Device:Buzzer
- added D1: LED_RGBA, LED_THT:LED_D5.0mm-4_RGB_Wide_Pins, symbol Device:LED_RGBA
Connections:
- net GND: now also BZ1.2 (-), D1.4 (A)
- net LED_R: now reaches U1.20 (GPIO6)
- net LED_R: now also D1.1 (RK)
- net LED_G: now reaches U1.21 (GPIO7)
- net LED_G: now also D1.2 (GK)
- net LED_B: now reaches U1.22 (GPIO8)
- net LED_B: now also D1.3 (BK)
- net BUZZER: now reaches U1.24 (GPIO2)
- net BUZZER: now also BZ1.1 (+)
Other:
- note added: "ESP32 38pin dev board"
- note added: "Indicators - LED and Buzzer"
- note added: "MPU6050 6dof sensor"
- note added: "Motor output terminal blocks"
- note added: "PWM Motor drivers"
- moved on the sheet: J2, J3, J4, J5, Q1, Q2, Q3, Q4, R1, R2, R3, R4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

Commit message: Lark1 refining
Parts:
- added D2: D, Diode_SMD:D_SOD-523, symbol Diode:1N4148WT
- added D3, D? (x3): D, symbol Device:D
Connections:
- net +3.3V: now also D3.1 (K), D?.1 (K), D?.1 (K), D?.1 (K)
- net M1_GND: now also D3.2 (A)
- net M2_GND: now also D?.2 (A)
- net M3_GND: now also D?.2 (A)
- net M4_GND: now also D?.2 (A)
- net at SW1.2 (B): now also D2.1 (K); no longer J1.2 (Pin_2)
- new net: D2.2 (A), J1.2 (Pin_2)
Other:
- moved on the sheet: J1

Commit message: Lark1 Kicad ERC check - no errors
Parts:
- gave numbers to parts that had none: 3
Connections:
- no-connect marks 1 -> 30
Other:
- note added: "Lark1 - Drone Flight Computer"
- moved on the sheet: BZ1, D1, D2, D3, D4, D5, D6, J1, J2, J3, J4, J5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
