File: Lark Flight computer/Lark1/Lark1.kicad_sch (KiCad schematic)
At the start: 23 parts, among them J1 Screw_Terminal_01x02, J2 Screw_Terminal_01x02, J3 Screw_Terminal_01x02, J4 Screw_Terminal_01x02, J5 Screw_Terminal_01x02, Q1 IRLZ44N, Q2 IRLZ44N, Q3 IRLZ44N, Q4 IRLZ44N, SW1 SW_SPDT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

Commit message: LarkOS1 started
Parts:
- removed D2: D, Diode_SMD:D_SOD-523, symbol Diode:1N4148WT
- added D2: D, Diode_THT:D_5KPW_P12.70mm_Horizontal, symbol Device:D
- added D7: LED, LED_THT:LED_D3.0mm, symbol Device:LED
- added R5: R, Resistor_THT:R_Axial_DIN0204_L3.6mm_D1.6mm_P5.08mm_Horizontal, symbol Device:R
- BZ1: footprint (none) -> Buzzer_Beeper:Buzzer_12x9.5RM7.6
- D3, D4, D5, D6: footprint (none) -> Diode_THT:D_5KPW_P12.70mm_Horizontal
- J1-BATT1: renamed from J1; footprint (none) -> TerminalBlock:TerminalBlock_Altech_AK300-2_P5.00mm
- J2-M1: renamed from J2; footprint (none) -> TerminalBlock:TerminalBlock_Altech_AK300-2_P5.00mm
- J3-M2: renamed from J3; footprint (none) -> TerminalBlock:TerminalBlock_Altech_AK300-2_P5.00mm
- J4-M3: renamed from J4; footprint (none) -> TerminalBlock:TerminalBlock_Altech_AK300-2_P5.00mm
- J5-M4: renamed from J5; footprint (none) -> TerminalBlock:TerminalBlock_Altech_AK300-2_P5.00mm
- R1, R2, R3, R4: footprint (none) -> Resistor_THT:R_Axial_DIN0204_L3.6mm_D1.6mm_P5.08mm_Horizontal
- U1: footprint esp32_lora_v2:esp32_devkitv4_38pin -> Connector_PinSocket_2.54mm:PinSocket_2x19_P2.54mm_Vertical
- U2: footprint usini_sensors:module_mpu6050 -> Connector_PinSocket_2.54mm:PinSocket_1x08_P2.54mm_Vertical
Connections:
- net +3.3V: now also R5.2
- net GND: now also D7.1 (K)
- net M1_PWM: now also U1.11 (GPIO27); no longer U1.31 (GPIO19)
- net M2_PWM: now also U1.12 (GPIO14); no longer U1.30 (GPIO18)
- net M3_PWM: now also U1.13 (GPIO12); no longer U1.29 (GPIO5)
- net M4_PWM: now also U1.15 (GPIO13); no longer U1.28 (GPIO17)
- net MPU6050_SCL: now also U1.10 (GPIO26); no longer U1.36 (GPIO22)
- net MPU6050_SDA: now also U1.9 (GPIO25); no longer U1.33 (GPIO21)
- net at SW1.2 (B): now also D2.1 (K)
- net at J1-BATT1.2 (Pin_2): now also D2.2 (A)
- new net: D7.2 (A), R5.1
- no-connect marks 30 -> 26
